File: CAN.kicad_sch (KiCad schematic)
At the start: 11 parts, among them SW3 SW_DIP_x05, U9 MCP2562-E-SN

Commit message: test
Connections:
- net FDCAN1_RX renamed RX
- net FDCAN1_TX renamed TX
Changed lines of the file:
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@@
 		)
 	)
-	(label "FDCAN1_RX"
+	(label "RX"
 		(at 129.54 107.95 0)
 		(effects
@@
 		)
 	)
-	(label "FDCAN1_TX"
+	(label "TX"
 		(at 129.54 105.41 0)
 		(effects
@@
 		)
 	)
-	(hierarchical_label "FDCAN1_RX"
+	(hierarchical_label "RX"
 		(shape input)
 		(at 129.54 107.95 180)
@@
 		)
 	)
-	(hierarchical_label "FDCAN1_TX"
+	(hierarchical_label "TX"
 		(shape output)
 		(at 129.54 105.41 180)
