File: MCU.kicad_sch (KiCad schematic)
At the start: 15 parts, among them J4 FTSH-107-01-L-D-K, SW2 SW_Push, U6 STM32G431KBTx, Y2 Crystal

Commit message: test
Connections:
- net CAN_ID_0: now reaches U6.10 (PA5)
- net CAN_ID_1: now reaches U6.11 (PA6)
- net CAN_ID_2: now reaches U6.12 (PA7)
- net CAN_ID_3: now reaches U6.18 (PA8)
Changed lines of the file:
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@@
+	(wire
+		(pts
+			(xy 167.64 102.87) (xy 179.07 102.87)
+		)
+		(stroke
+			(width 0)
+			(type default)
+		)
+	)
 	(wire
 		(pts
@@
 	(wire
 		(pts
+			(xy 167.64 100.33) (xy 179.07 100.33)
+		)
+		(stroke
+			(width 0)
+			(type default)
+		)
+	)
+	(wire
+		(pts
 			(xy 115.57 53.34) (xy 115.57 54.61)
 		)
@@
 	(wire
 		(pts
+			(xy 167.64 95.25) (xy 179.07 95.25)
+		)
+		(stroke
+			(width 0)
+			(type default)
+		)
+	)
+	(wire
+		(pts
 			(xy 115.57 53.34) (xy 125.73 53.34)
 		)
@@
 		(pts
 			(xy 210.82 60.96) (xy 207.01 60.96)
+		)
+		(stroke
+			(width 0)
+			(type default)
+		)
+	)
+	(wire
+		(pts
+			(xy 167.64 97.79) (xy 179.07 97.79)
 		)
 		(stroke
@@
 		)
 	)
+	(label "CAN_ID_1"
+		(at 179.07 97.79 180)
+		(effects
+			(font
+				(size 1.27 1.27)
+			)
+			(justify right bottom)
+		)
+	)
 	(label "NRST"
 		(at 137.16 82.55 0)
@@
 		)
 	)
+	(label "CAN_ID_0"
+		(at 179.07 95.25 180)
+		(effects
+			(font
+				(size 1.27 1.27)
+			)
+			(justify right bottom)
+		)
+	)
 	(label "SWCLK"
 		(at 179.07 118.11 180)
@@
 		)
 	)
+	(label "CAN_ID_2"
+		(at 179.07 100.33 180)
+		(effects
+			(font
+				(size 1.27 1.27)
+			)
+			(justify right bottom)
+		)
+	)
 	(label "FDCAN1_TX"
 		(at 179.07 113.03 180)
@@
 		)
 	)
+	(label "CAN_ID_3"
+		(at 179.07 102.87 180)
+		(effects
+			(font
+				(size 1.27 1.27)
+			)
+			(justify right bottom)
+		)
+	)
+	(hierarchical_label "CAN_ID_2"
+		(shape input)
+		(at 179.07 100.33 0)
+		(effects
+			(font
+				(size 1.27 1.27)
+			)
+			(justify left)
+		)
+	)
+	(hierarchical_label "CAN_ID_3"
+		(shape input)
+		(at 179.07 102.87 0)
+		(effects
+			(font
+				(size 1.27 1.27)
+			)
+			(justify left)
+		)
+	)
+	(hierarchical_label "CAN_ID_0"
+		(shape input)
+		(at 179.07 95.25 0)
+		(effects
+			(font
+				(size 1.27 1.27)
+			)
+			(justify left)
+		)
+	)
+	(hierarchical_label "CAN_ID_1"
+		(shape input)
+		(at 179.07 97.79 0)
+		(effects
+			(font
+				(size 1.27 1.27)
+			)
+			(justify left)
+		)
+	)
