File: Stepper.kicad_sch (KiCad schematic)
At the start: 3 parts, among them U5 TMC2209_SILENTSTEPSTICK

Commit message: test
Parts:
- removed U5: TMC2209_SILENTSTEPSTICK, Library:MODULE_TMC2209_SILENTSTEPSTICK, symbol Library:TMC2209_SILENTSTEPSTICK
- added C26, C30: 100nF, symbol Device:C
- added C27: 100uF, symbol Device:C_Polarized
- added C28, C29, C32: 0.1uF, symbol Device:C
- added C31: 22nF, symbol Device:C
- added R10, R11: 20K, symbol Device:R
- added R8, R9: 0.05R, symbol Device:R
- added RV1: 10K, symbol Device:R_Potentiometer
- added U5: TMC2209-LA, Package_DFN_QFN:VQFN-28-1EP_5x5mm_P0.5mm_EP3.7x3.7mm_ThermalVias, symbol Driver_Motor:TMC2209-LA
- R12, R13: value 10K -> 20K; footprint Resistor_SMD:R_0603_1608Metric -> (none)
Connections:
- net +3V3: now also C30.1, C32.1, R10.1, U5.15 (VCC_IO); no longer R12.1
- net DIR: now also U5.19 (DIR)
- net EN: now also R13.1, U5.2 (~{EN})
- net GND: now also R12.2, R13.2, C27.2, C28.2, C29.2, C30.2, C32.2, R8.2, R9.2, RV1.3, U5.13 (CLK), U5.18 (GND), U5.25 (NC), U5.29 (GND), U5.3 (GND); no longer R13.1
- net MS1: now also U5.9 (MS1/AD0); no longer R13.2
- net MS2: now also U5.10 (MS2/AD1); no longer R12.2
- net STEP: now also R12.1, U5.16 (STEP)
- new net: RV1.2, U5.17 (VREF)
- new net: R9.1, U5.23 (BRA)
- new net: R8.1, U5.27 (BRB)
- new net: C31.2, U5.4 (CPO)
- new net: C31.1, U5.5 (CPI)
- new net: C26.2, U5.6 (VCP)
- new net: R10.2, RV1.1
- new net +12V: C26.1, C27.1, C28.1, C29.1, U5.22 (VS), U5.28 (VS)
- new net 5VOUT: U5.8 (5VOUT)
- new net OA1: U5.24 (OA1)
- new net OA2: U5.21 (OA2)
- new net OB1: U5.26 (OB1)
- new net OB2: U5.1 (OB2)
- new net RX: R11.1
- new net SPREAD: U5.7 (SPREAD)
- new net TX: R11.2, U5.14 (~{PD}/UART)
- no-connect marks 4 -> 3
