File: Syringe-Pump-Driver.kicad_pcb (KiCad board)
At the start: 2 copper layers, 37 x 25.5 mm, 40 parts, among them J1 USB_C_Receptacle_USB2.0_16P, J3 Conn_01x02, SW1 SW_Push, U1 ATmega328P-A, U2 FT232RL, U3 TPD2EUSB30, U4 MAX40200AUK, U5 TMC2209_SILENTSTEPSTICK, U7 MAX40200AUK, U8 NCP718xSN500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

Commit message: Updated
Parts:
- removed C1: 100nF, Capacitor_SMD:C_0603_1608Metric
- removed C6: 1uF, Capacitor_SMD:C_0603_1608Metric
- removed C7: 10uF, Capacitor_SMD:C_0603_1608Metric
- removed H1, H2: MountingHole_Pad, Connector_Wire:SolderWirePad_1x01_SMD_3x6mm
- removed H10, H5: MountingHole_Pad, TestPoint:TestPoint_THTPad_D1.0mm_Drill0.5mm
- removed H12: MountingHole, MountingHole:MountingHole_2.2mm_M2_DIN965_Pad_TopBottom
- removed H3, H4, H6, H7, H8, H9: MountingHole_Pad, Connector_Wire:SolderWirePad_1x01_SMD_2x4mm
- removed J3: Conn_01x02, Connector_JST:JST_PH_B2B-PH-K_1x02_P2.00mm_Vertical
- removed R1, R2, R7, R8: 1K, Resistor_SMD:R_0603_1608Metric
- removed SW1: SW_Push, Button_Switch_SMD:SW_SPST_FSMSM
- removed Y1: Resonator, Crystal:Resonator_SMD_Murata_CSTxExxV-3Pin_3.0x1.1mm_HandSoldering
- added C125: 0.1uF, Capacitor_SMD:C_0805_2012Metric, F.Cu at (-27.8, 25.6)
- added C14: 1uF, Capacitor_SMD:C_0603_1608Metric, F.Cu at (-27.8, 13.9)
- added C15: 1uF, Capacitor_SMD:C_0603_1608Metric, F.Cu at (-27.8, 16.4)
- added C24: 1uF, Capacitor_SMD:C_0603_1608Metric, F.Cu at (-62.5, 47.8)
- added C25: 1uF, Capacitor_SMD:C_0603_1608Metric, F.Cu at (-62.5, 50.3)
- added J4: FTSH-107-01-L-D-K, Connector_Samtec:SAMTEC_FTSH-107-01-L-D-K, F.Cu at (-35.2, 27.4)
- added U10: MCP1700x-150xxTT, Package_TO_SOT_SMD:SOT-23, F.Cu at (-52.9, 47.1)
- added U6: STM32G431KBTx, Package_QFP:LQFP-32_7x7mm_P0.8mm, F.Cu at (-35.5, 18.3)
- added U9: MCP2562-E-SN, Package_SO:SOIC-8_3.9x4.9mm_P1.27mm, F.Cu at (-26.6, 53.6)
- C5: value 10uF -> 1uF
- C8, C9, F1, R5, R6, U2, U3, U7: moved to F.Cu
- R12, R13: value 1K -> 10K; moved to F.Cu
- U1: value ATmega328P-A -> LD1117S50TR_SOT223; footprint Package_QFP:TQFP-32_7x7mm_P0.8mm -> Package_TO_SOT_SMD:SOT-223-3_TabPin2
- U8: value NCP718xSN500 -> AP2127K-3.3; moved to F.Cu
- moved C4 239.6 mm to (-62.5, 37.8), turned to 0 degrees
- moved C5 238.0 mm to (-62.5, 40.3), turned to 0 degrees
- moved U1 225.2 mm to (-55.6, 40.7)
- moved U4 217.5 mm to (-45.9, 49.0), turned to 0 degrees
- moved J1 212.2 mm to (-42.6, 41.9), turned to 0 degrees
- moved U5 211.9 mm to (-55.6, 23.6), turned to 180 degrees
- moved C3 210.5 mm to (-34.8, 40.3), turned to 0 degrees
- moved R13 210.0 mm to (-45.3, 16.4)
- moved R12 210.0 mm to (-45.3, 13.9)
- moved C9 209.4 mm to (-62.5, 45.3), turned to 0 degrees
- moved C8 209.1 mm to (-62.5, 42.8), turned to 0 degrees
- moved F1 208.3 mm to (-41.1, 48.1), turned to 0 degrees
- moved U7 207.2 mm to (-58.0, 47.2)
- moved C2 206.1 mm to (-34.8, 37.8)
- moved U8 203.3 mm to (-58.0, 51.9), turned to 0 degrees
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Connections:
- net /MS1 renamed /Stepper Driver/MS1
- net /MS2 renamed /Stepper Driver/MS2
- net Net-(U2-USBD+) renamed /USB-UART/D+
- net Net-(U2-USBD-) renamed /USB-UART/D-
- C5 pad 2: +5V -> +3V3
- C8 pad 2: +24V -> +12V
- C9 pad 2: Net-(U7-EN) -> Net-(U1-VO)
- R12 pad 1: +5V -> +3V3
- U1 pad 1: /DIR -> GND
- U1 pad 2: /STEP -> Net-(U1-VO)
- U1 pad 3: GND -> +12V
- U2 pad 1: /RX -> /MCU/USART1_RX
- U2 pad 2: Net-(U2-DTR) -> unconnected-(U2-DTR-Pad2)
- U2 pad 4: +5V -> +3V3
- U2 pad 5: /TX -> /MCU/USART1_TX
- U5 pad 10: /STEP -> /Stepper Driver/STEP
- U5 pad 12: /UART -> /Stepper Driver/UART
- U5 pad 16: /EN -> /Stepper Driver/EN
- U5 pad 2: +5V -> +3V3
- U5 pad 3: Net-(U5-M1B) -> unconnected-(U5-M1B-Pad3)
- U5 pad 4: Net-(U5-M1A) -> unconnected-(U5-M1A-Pad4)
- U5 pad 5: Net-(U5-M2A) -> unconnected-(U5-M2A-Pad5)
- U5 pad 6: Net-(U5-M2B) -> unconnected-(U5-M2B-Pad6)
- U5 pad 9: /DIR -> /Stepper Driver/DIR
- U7 pad 1: Net-(U7-EN) -> Net-(U1-VO)
- U7 pad 3: Net-(U7-EN) -> Net-(U1-VO)
- U8 pad 1: +24V -> +5V
- U8 pad 3: +24V -> +5V
- U8 pad 5: Net-(U7-EN) -> +3V3
Routing:
- net +5V: track 55.0 -> 0.00 mm, vias 9 -> 0
- net /ESTOP: track 30.0 -> 0.00 mm, vias 1 -> 0
- net /RESET: track 24.9 -> 0.00 mm, vias 3 -> 0
- net /UART: track 19.0 -> 0.00 mm, vias 2 -> 0
- net /USB-UART/D-: track 17.9 -> 0.00 mm, vias 1 -> 0
- net /DIR: track 17.5 -> 0.00 mm
- net /SCL: track 16.7 -> 0.00 mm
- net /USB-UART/D+: track 16.3 -> 0.00 mm, vias 1 -> 0
- net /STEP: track 16.3 -> 0.00 mm
- net /SDA: track 15.8 -> 0.00 mm
- net /EN: track 14.3 -> 0.00 mm, vias 1 -> 0
- net Net-(U1-PD0): track 8.68 -> 0.00 mm, vias 1 -> 0
- net /RX: track 7.99 -> 0.00 mm
- net Net-(U1-PD1): track 7.80 -> 0.00 mm, vias 1 -> 0
- net Net-(U4-EN): track 6.86 -> 0.00 mm, vias 2 -> 0
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- removed copper zone on B.Cu, net +24V
- removed copper zone on F.Cu, net +24V
- removed copper zone on B.Cu, net +5V
- removed copper zone on F.Cu, net +5V
- removed copper zone on F.Cu, net /USB-UART/D+
- removed copper zone on B.Cu, net GND
- removed copper zone on F.Cu, net GND
- removed copper zone on F.Cu, net Net-(F1-Pad1)
- removed copper zone on F.Cu, net Net-(U4-EN)
- removed copper zone on B.Cu, net Net-(U7-EN)
Other:
- board outline removed

Commit message: test
Parts:
- removed R12, R13: 10K, Resistor_SMD:R_0603_1608Metric
- U5: value TMC2209_SILENTSTEPSTICK -> TMC2209-LA; footprint Library:MODULE_TMC2209_SILENTSTEPSTICK -> Package_DFN_QFN:VQFN-28-1EP_5x5mm_P0.5mm_EP3.7x3.7mm_ThermalVias
- moved U5 1.65 mm to (-56.7, 22.3), turned to 0 degrees
Connections:
- net +24V renamed /Stepper Driver/5VOUT
- U5 pad 1: GND -> unconnected-(U5-OB2-Pad1)
- U5 pad 10: /Stepper Driver/STEP -> unconnected-(U5-MS2/AD1-Pad10)
- U5 pad 12: /Stepper Driver/UART -> unconnected-(U5-INDEX-Pad12)
- U5 pad 13: unconnected-(U5-SPRD-Pad13) -> GND
- U5 pad 14: /Stepper Driver/MS2 -> unconnected-(U5-~{PD}/UART-Pad14)
- U5 pad 15: /Stepper Driver/MS1 -> +3V3
- U5 pad 16: /Stepper Driver/EN -> unconnected-(U5-STEP-Pad16)
- U5 pad 17: unconnected-(U5-INDEX-Pad17) -> Net-(U5-VREF)
- U5 pad 18: unconnected-(U5-DIAG-Pad18) -> GND
- U5 pad 2: +3V3 -> unconnected-(U5-~{EN}-Pad2)
- U5 pad 3: unconnected-(U5-M1B-Pad3) -> GND
- U5 pad 4: unconnected-(U5-M1A-Pad4) -> Net-(U5-CPO)
- U5 pad 5: unconnected-(U5-M2A-Pad5) -> Net-(U5-CPI)
- U5 pad 6: unconnected-(U5-M2B-Pad6) -> Net-(U5-VCP)
- U5 pad 7: GND -> unconnected-(U5-SPREAD-Pad7)
- U5 pad 9: /Stepper Driver/DIR -> unconnected-(U5-MS1/AD0-Pad9)
- U6 pad 10: unconnected-(U6-PA5-Pad10) -> /CAN/CAN_ID_0
- U6 pad 11: unconnected-(U6-PA6-Pad11) -> /CAN/CAN_ID_1
- U6 pad 12: unconnected-(U6-PA7-Pad12) -> /CAN/CAN_ID_2
- U6 pad 18: unconnected-(U6-PA8-Pad18) -> /CAN/CAN_ID_3
