File: Syringe-Pump-Driver.kicad_sch (KiCad schematic)
At the start: 40 parts, among them J1 USB_C_Receptacle_USB2.0_16P, J3 Conn_01x02, SW1 SW_Push, U1 ATmega328P-A, U2 FT232RL, U3 TPD2EUSB30, U4 MAX40200AUK, U5 TMC2209_SILENTSTEPSTICK, U7 MAX40200AUK, U8 NCP718xSN500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

Commit message: Updated
Parts:
- removed C1: 100nF, Capacitor_SMD:C_0603_1608Metric, symbol Device:C
- removed C2, C3, C4, C6, C8, C9: 1uF, Capacitor_SMD:C_0603_1608Metric, symbol Device:C
- removed C5, C7: 10uF, Capacitor_SMD:C_0603_1608Metric, symbol Device:C
- removed F1: 500mA, Fuse:Fuse_0805_2012Metric, symbol Device:Fuse
- removed H1, H2: MountingHole_Pad, Connector_Wire:SolderWirePad_1x01_SMD_3x6mm, symbol Mechanical:MountingHole_Pad
- removed H10, H5: MountingHole_Pad, TestPoint:TestPoint_THTPad_D1.0mm_Drill0.5mm, symbol Mechanical:MountingHole_Pad
- removed H12: MountingHole, MountingHole:MountingHole_2.2mm_M2_DIN965_Pad_TopBottom, symbol Mechanical:MountingHole
- removed H3, H4, H6, H7, H8, H9: MountingHole_Pad, Connector_Wire:SolderWirePad_1x01_SMD_2x4mm, symbol Mechanical:MountingHole_Pad
- removed J1: USB_C_Receptacle_USB2.0_16P, Connector_USB:USB_C_Receptacle_G-Switch_GT-USB-7010ASV, symbol Connector:USB_C_Receptacle_USB2.0_16P
- removed J3: Conn_01x02, Connector_JST:JST_PH_B2B-PH-K_1x02_P2.00mm_Vertical, symbol Connector_Generic:Conn_01x02
- removed R1, R12, R13, R2, R7, R8: 1K, Resistor_SMD:R_0603_1608Metric, symbol Device:R
- removed R5, R6: 5.1K, Resistor_SMD:R_0603_1608Metric, symbol Device:R
- removed SW1: SW_Push, Button_Switch_SMD:SW_SPST_FSMSM, symbol Switch:SW_Push
- removed U1: ATmega328P-A, Package_QFP:TQFP-32_7x7mm_P0.8mm, symbol MCU_Microchip_ATmega:ATmega328P-A
- removed U2: FT232RL, Package_SO:SSOP-28_5.3x10.2mm_P0.65mm, symbol Interface_USB:FT232RL
- removed U3: TPD2EUSB30, Package_TO_SOT_SMD:Texas_DRT-3, symbol Power_Protection:TPD2EUSB30
- removed U4, U7: MAX40200AUK, Package_TO_SOT_SMD:SOT-23-5, symbol Analog_Switch:MAX40200AUK
- removed U5: TMC2209_SILENTSTEPSTICK, Library:MODULE_TMC2209_SILENTSTEPSTICK, symbol Library:TMC2209_SILENTSTEPSTICK
- removed U8: NCP718xSN500, Package_TO_SOT_SMD:SOT-23-5, symbol Regulator_Linear:NCP718xSN500
- removed Y1: Resonator, Crystal:Resonator_SMD_Murata_CSTxExxV-3Pin_3.0x1.1mm_HandSoldering, symbol Device:Resonator
Connections:
- no-connect marks 32 -> 0
Other:
- added sheet CAN (CAN.kicad_sch)
- added sheet MCU (MCU.kicad_sch)
- added sheet Power (Power.kicad_sch)
- added sheet Stepper Driver (Stepper.kicad_sch)
- added sheet USB (USB.kicad_sch)
- added sheet USB-UART (USB-UART.kicad_sch)

Commit message: test
Other:
- sheet CAN ports: added RX, TX; removed FDCAN1_RX, FDCAN1_TX
- sheet MCU ports: added CAN_ID_0, CAN_ID_1, CAN_ID_2, CAN_ID_3; removed none
- sheet Stepper Driver ports: added EN, RX, STEP, TX; removed none
- sheet USB-UART ports: added RX, TX; removed USART1_RX, USART1_TX
Changed lines of the file:
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@@
+	(wire
+		(pts
+			(xy 175.26 81.28) (xy 181.61 81.28)
+		)
+		(stroke
+			(width 0)
+			(type default)
+		)
+	)
 	(wire
 		(pts
 			(xy 92.71 69.85) (xy 105.41 69.85)
+		)
+		(stroke
+			(width 0)
+			(type default)
+		)
+	)
+	(wire
+		(pts
+			(xy 175.26 76.2) (xy 181.61 76.2)
+		)
+		(stroke
+			(width 0)
+			(type default)
+		)
+	)
+	(wire
+		(pts
+			(xy 175.26 78.74) (xy 181.61 78.74)
+		)
+		(stroke
+			(width 0)
+			(type default)
+		)
+	)
+	(wire
+		(pts
+			(xy 175.26 73.66) (xy 181.61 73.66)
 		)
 		(stroke
@@
 			)
 		)
+		(pin "CAN_ID_0" input
+			(at 175.26 73.66 0)
+			(effects
+				(font
+					(size 1.27 1.27)
+				)
+				(justify right)
+			)
+		)
+		(pin "CAN_ID_1" input
+			(at 175.26 76.2 0)
+			(effects
+				(font
+					(size 1.27 1.27)
+				)
+				(justify right)
+			)
+		)
+		(pin "CAN_ID_2" input
+			(at 175.26 78.74 0)
+			(effects
+				(font
+					(size 1.27 1.27)
+				)
+				(justify right)
+			)
+		)
+		(pin "CAN_ID_3" input
+			(at 175.26 81.28 0)
+			(effects
+				(font
+					(size 1.27 1.27)
+				)
+				(justify right)
+			)
+		)
 		(instances
 			(project "Syringe-Pump-Driver"
@@
 			)
 		)
-		(pin "USART1_RX" output
+		(pin "RX" input
 			(at 124.46 67.31 0)
 			(effects
@@
 			)
 		)
-		(pin "USART1_TX" input
+		(pin "TX" output
 			(at 124.46 69.85 0)
 			(effects
@@
 			)
 		)
-		(pin "FDCAN1_RX" input
+		(pin "RX" input
 			(at 181.61 67.31 180)
 			(effects
@@
 			)
 		)
-		(pin "FDCAN1_TX" output
+		(pin "TX" output
 			(at 181.61 69.85 180)
 			(effects
@@
 			)
 		)
+		(pin "EN" input
+			(at 181.61 97.79 180)
+			(effects
+				(font
+					(size 1.27 1.27)
+				)
+				(justify left)
+			)
+		)
+		(pin "RX" input
+			(at 181.61 104.14 180)
+			(effects
+				(font
+					(size 1.27 1.27)
+				)
+				(justify left)
+			)
+		)
+		(pin "STEP" input
+			(at 181.61 100.33 180)
+			(effects
+				(font
+					(size 1.27 1.27)
+				)
+				(justify left)
+			)
+		)
+		(pin "TX" output
+			(at 181.61 106.68 180)
+			(effects
+				(font
+					(size 1.27 1.27)
+				)
+				(justify left)
+			)
+		)
