File: USB-UART.kicad_sch (KiCad schematic)
At the start: 5 parts, among them U2 FT232RL

Commit message: test
Connections:
- net USART1_RX renamed TX
- net USART1_TX renamed RX
Changed lines of the file:
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@@
 		)
 	)
-	(label "USART1_TX"
+	(label "RX"
 		(at 179.07 90.17 180)
 		(effects
@@
 		)
 	)
-	(label "USART1_RX"
+	(label "TX"
 		(at 179.07 87.63 180)
 		(effects
@@
 		)
 	)
-	(hierarchical_label "USART1_TX"
+	(hierarchical_label "RX"
 		(shape input)
 		(at 179.07 90.17 0)
@@
 		)
 	)
-	(hierarchical_label "USART1_RX"
+	(hierarchical_label "TX"
 		(shape output)
 		(at 179.07 87.63 0)
